File: mx/pcb/qapla_mx/qapla_mx.kicad_pcb (KiCad board)
At the start: 2 copper layers, 164.2 x 137.2 mm, 72 parts

Commit message: Routing MX switches
Parts:
- removed _1: , reset_switch
- removed _2: , switch_JS102011SAQN
- removed _3: , D_0805_2012Metric_Pad1.15x1.40mm_HandSolder
- removed _3: , R_0805_2012Metric_Pad1.20x1.40mm_HandSolder
- added REF**: VIA-0.6mm, VIA-0.6mm, F.Cu at (216.3, 67.9)
- added REF**: VIA-0.6mm, VIA-0.6mm, F.Cu at (197.3, 26.4)
- added REF**: VIA-0.6mm, VIA-0.6mm, F.Cu at (155.9, 67.2)
- added REF**: VIA-0.6mm, VIA-0.6mm, F.Cu at (178.3, 22.4)
- added REF**: VIA-0.6mm, VIA-0.6mm, F.Cu at (109.9, 47.7)
- added REF**: VIA-0.6mm, VIA-0.6mm, F.Cu at (119.8, 103.8)
- added REF**: VIA-0.6mm, VIA-0.6mm, F.Cu at (216.3, 85.9)
- added REF**: VIA-0.6mm, VIA-0.6mm, F.Cu at (155.8, 66.2)
- added REF**: VIA-0.6mm, VIA-0.6mm, F.Cu at (116.7, 86.1)
- added REF**: VIA-0.6mm, VIA-0.6mm, F.Cu at (178.3, 21.4)
- added REF**: VIA-0.6mm, VIA-0.6mm, F.Cu at (197.3, 65.4)
- added REF**: VIA-0.6mm, VIA-0.6mm, F.Cu at (116.5, 85.1)
- added REF**: VIA-0.6mm, VIA-0.6mm, F.Cu at (178.3, 78.4)
- added REF**: VIA-0.6mm, VIA-0.6mm, F.Cu at (157.5, 85.1)
- added REF**: VIA-0.6mm, VIA-0.6mm, F.Cu at (135.2, 81.8)
- added REF**: VIA-0.6mm, VIA-0.6mm, F.Cu at (135.4, 82.8)
- added REF**: VIA-0.6mm, VIA-0.6mm, F.Cu at (238.6, 133.1)
- added REF**: VIA-0.6mm, VIA-0.6mm, F.Cu at (235.3, 88.4)
- added REF**: VIA-0.6mm, VIA-0.6mm, F.Cu at (197.3, 64.4)
- added REF**: VIA-0.6mm, VIA-0.6mm, F.Cu at (152.5, 28.3)
- added REF**: VIA-0.6mm, VIA-0.6mm, F.Cu at (131.9, 63.1)
- added REF**: VIA-0.6mm, VIA-0.6mm, F.Cu at (113.2, 66.4)
- added REF**: VIA-0.6mm, VIA-0.6mm, F.Cu at (154.1, 47.2)
- added REF**: VIA-0.6mm, VIA-0.6mm, F.Cu at (216.3, 66.9)
- added REF**: VIA-0.6mm, VIA-0.6mm, F.Cu at (178.3, 40.4)
- added REF**: VIA-0.6mm, VIA-0.6mm, F.Cu at (216.3, 29.9)
- added REF**: VIA-0.6mm, VIA-0.6mm, F.Cu at (178.3, 59.4)
- added REF**: VIA-0.6mm, VIA-0.6mm, F.Cu at (152.6, 29.3)
- added REF**: VIA-0.6mm, VIA-0.6mm, F.Cu at (128.6, 44.4)
- added REF**: VIA-0.6mm, VIA-0.6mm, F.Cu at (178.3, 97.4)
- added REF**: VIA-0.6mm, VIA-0.6mm, F.Cu at (216.3, 47.9)
- added REF**: VIA-0.6mm, VIA-0.6mm, F.Cu at (203.6, 110.0)
- added REF**: VIA-0.6mm, VIA-0.6mm, F.Cu at (110.1, 48.7)
- added REF**: VIA-0.6mm, VIA-0.6mm, F.Cu at (197.3, 45.4)
- added REF**: VIA-0.6mm, VIA-0.6mm, F.Cu at (138.5, 100.5)
- added REF**: VIA-0.6mm, VIA-0.6mm, F.Cu at (216.3, 28.9)
- added REF**: VIA-0.6mm, VIA-0.6mm, F.Cu at (220.1, 121.9)
- added REF**: VIA-0.6mm, VIA-0.6mm, F.Cu at (197.3, 83.4)
- added REF**: VIA-0.6mm, VIA-0.6mm, F.Cu at (197.3, 27.4)
- added REF**: VIA-0.6mm, VIA-0.6mm, F.Cu at (128.8, 45.4)
- added REF**: VIA-0.6mm, VIA-0.6mm, F.Cu at (178.3, 60.4)
- added _42: , reset_switch, F.Cu at (252.8, 55.9)
- added _43: , switch_JS102011SAQN, F.Cu at (251.6, 28.4)
- added _44: , R_0805_2012Metric_Pad1.20x1.40mm_HandSolder, F.Cu at (237.8, 67.7)
- added _44: , D_0805_2012Metric_Pad1.15x1.40mm_HandSolder, F.Cu at (237.8, 67.7)
- moved D27 0.13 mm to (210.9, 111.6)
- moved D19 0.13 mm to (185.8, 97.1)
- moved D20 0.13 mm to (185.8, 78.1)
- moved D25 0.13 mm to (223.8, 47.6)
- moved D24 0.13 mm to (223.8, 85.6)
- moved D23 0.13 mm to (204.8, 45.1)
- moved D26 0.13 mm to (242.8, 88.1)
- moved D22 0.13 mm to (204.8, 83.1)
- moved D21 0.13 mm to (185.8, 40.1)
- moved D17 0.12 mm to (164.9, 84.2)
- moved D18 0.12 mm to (161.6, 46.3)
- moved D13 0.12 mm to (127.1, 102.2)
- moved D14 0.12 mm to (120.5, 64.8)
- moved D15 0.12 mm to (145.8, 98.9)
- moved D16 0.12 mm to (139.2, 61.5)
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Routing:
- net (no net): track 337.7 -> 0.00 mm
- net P16: track 0.00 -> 204.2 mm
- net P15: track 0.00 -> 187.6 mm
- net P14: track 0.00 -> 168.6 mm
- net P18: track 0.00 -> 148.6 mm
- net P20: track 0.00 -> 147.6 mm
- net P6: track 0.00 -> 146.0 mm
- net P8: track 0.00 -> 130.9 mm
- net P9: track 0.00 -> 130.1 mm
- net P19: track 0.00 -> 128.2 mm
- net P7: track 0.00 -> 125.0 mm
- net P10: track 0.00 -> 93.8 mm
- net P5: track 0.00 -> 77.2 mm
- net GND: track 0.00 -> 29.5 mm
- net middle_num: track 0.00 -> 27.1 mm
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Other:
- outline, holes or cut-outs redrawn

Commit message: Finalizing Qapla MX PCB
Parts:
- moved MH1 0.16 mm to (231.1, 82.4)
- moved S23 0.08 mm to (216.2, 74.9)
- moved S11 0.08 mm to (154.8, 55.2)
- moved _42 0.08 mm to (252.7, 55.9)
- moved D11 0.08 mm to (223.7, 83.2)
- moved D5 0.08 mm to (164.6, 81.8)
- moved REF** 0.08 mm to (197.2, 65.4)
- moved REF** 0.08 mm to (110.0, 48.7)
- moved JST1 0.08 mm to (251.5, 35.9)
- moved D18 0.08 mm to (161.5, 46.3)
- moved D9 0.08 mm to (204.7, 80.7)
- moved REF** 0.08 mm to (235.2, 88.4)
- moved _44 0.08 mm to (237.7, 67.7) (x2)
- moved REF** 0.08 mm to (197.2, 45.4)
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Connections:
- _44 pad 3: P4 -> P21
Routing:
- net P20: track 147.6 -> 289.9 mm
- net P19: track 128.2 -> 268.9 mm
- net GND: track 29.5 -> 121.2 mm, vias 0 -> 2
- net P18: track 148.6 -> 239.4 mm
- net P5: track 77.2 -> 167.0 mm, vias 0 -> 1
- net P14: track 168.6 -> 237.7 mm
- net P15: track 187.6 -> 251.1 mm
- net P1: track 9.83 -> 70.9 mm, vias 0 -> 1
- net P6: track 146.0 -> 204.5 mm, vias 0 -> 1
- net P8: track 130.9 -> 188.4 mm, vias 0 -> 1
- net P9: track 130.1 -> 186.0 mm, vias 0 -> 1
- net P7: track 125.0 -> 178.3 mm, vias 0 -> 1
- net P10: track 93.8 -> 137.1 mm, vias 0 -> 1
- net VCC: track 9.84 -> 50.8 mm
- net P2: track 9.83 -> 50.4 mm, vias 0 -> 1
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- added copper zone on B.Cu, net GND
- added copper zone on F.Cu, net GND

Commit message: MX Keyboard has a batleth
Parts:
- removed the REF** at (216.2, 67.9)
- removed the REF** at (197.2, 26.4)
- removed the REF** at (155.8, 67.2)
- removed the REF** at (178.2, 22.4)
- removed the REF** at (109.8, 47.7)
- removed the REF** at (119.7, 103.8)
- removed the REF** at (216.2, 85.9)
- removed the REF** at (155.7, 66.2)
- removed the REF** at (116.6, 86.1)
- removed the REF** at (178.2, 21.4)
- removed the REF** at (197.2, 65.4)
- removed the REF** at (116.4, 85.1)
- removed the REF** at (178.2, 78.4)
- removed the REF** at (157.4, 85.1)
- removed the REF** at (135.1, 81.8)
- removed the REF** at (135.3, 82.8)
- removed the REF** at (238.5, 133.1)
- removed the REF** at (235.2, 88.4)
- removed the REF** at (197.2, 64.4)
- removed the REF** at (152.4, 28.3)
- removed the REF** at (131.8, 63.1)
- removed the REF** at (113.1, 66.4)
- removed the REF** at (154.1, 47.3)
- removed the REF** at (216.2, 66.9)
- removed the REF** at (178.2, 40.4)
- removed the REF** at (216.2, 29.9)
- removed the REF** at (178.2, 59.4)
- removed the REF** at (152.5, 29.3)
- removed the REF** at (128.5, 44.4)
- removed the REF** at (178.2, 97.4)
- removed the REF** at (216.2, 47.9)
- removed the REF** at (203.5, 110.0)
- removed the REF** at (110.0, 48.7)
- removed the REF** at (197.2, 45.4)
- removed the REF** at (138.4, 100.5)
- removed the REF** at (216.2, 28.9)
- removed the REF** at (220.0, 121.9)
- removed the REF** at (197.2, 83.4)
- removed the REF** at (197.2, 27.4)
- removed the REF** at (128.7, 45.4)
- removed the REF** at (178.2, 60.4)
- removed the _44 at (237.7, 67.7) (x2)
- added ?: , footprints:batleth, F.Cu at (242.1, 77.1)
- added REF**: VIA-0.6mm, VIA-0.6mm, F.Cu at (128.6, 45.7)
- added REF**: VIA-0.6mm, VIA-0.6mm, F.Cu at (178.2, 40.7)
- added REF**: VIA-0.6mm, VIA-0.6mm, F.Cu at (216.2, 48.2)
- added REF**: VIA-0.6mm, VIA-0.6mm, F.Cu at (113.1, 66.7)
- added REF**: VIA-0.6mm, VIA-0.6mm, F.Cu at (238.5, 133.4)
- added REF**: VIA-0.6mm, VIA-0.6mm, F.Cu at (197.2, 45.7)
- added REF**: VIA-0.6mm, VIA-0.6mm, F.Cu at (203.5, 110.3)
- added REF**: VIA-0.6mm, VIA-0.6mm, F.Cu at (155.8, 67.5)
- added REF**: VIA-0.6mm, VIA-0.6mm, F.Cu at (135.1, 82.2)
- added REF**: VIA-0.6mm, VIA-0.6mm, F.Cu at (216.2, 86.2)
- added REF**: VIA-0.6mm, VIA-0.6mm, F.Cu at (135.2, 83.1)
- added REF**: VIA-0.6mm, VIA-0.6mm, F.Cu at (220.0, 122.3)
- added REF**: VIA-0.6mm, VIA-0.6mm, F.Cu at (157.3, 85.4)
- added REF**: VIA-0.6mm, VIA-0.6mm, F.Cu at (178.2, 78.7)
- added REF**: VIA-0.6mm, VIA-0.6mm, F.Cu at (216.2, 68.2)
- added REF**: VIA-0.6mm, VIA-0.6mm, F.Cu at (155.7, 66.5)
- added REF**: VIA-0.6mm, VIA-0.6mm, F.Cu at (116.4, 85.5)
- added REF**: VIA-0.6mm, VIA-0.6mm, F.Cu at (197.2, 65.7)
- added REF**: VIA-0.6mm, VIA-0.6mm, F.Cu at (109.8, 48.0)
- added REF**: VIA-0.6mm, VIA-0.6mm, F.Cu at (178.2, 21.7)
- added REF**: VIA-0.6mm, VIA-0.6mm, F.Cu at (178.2, 97.7)
- added REF**: VIA-0.6mm, VIA-0.6mm, F.Cu at (216.2, 29.2)
- added REF**: VIA-0.6mm, VIA-0.6mm, F.Cu at (216.2, 67.2)
- added REF**: VIA-0.6mm, VIA-0.6mm, F.Cu at (197.2, 27.7)
- added REF**: VIA-0.6mm, VIA-0.6mm, F.Cu at (116.5, 86.4)
- added REF**: VIA-0.6mm, VIA-0.6mm, F.Cu at (154.0, 47.6)
- added REF**: VIA-0.6mm, VIA-0.6mm, F.Cu at (152.4, 28.7)
- added REF**: VIA-0.6mm, VIA-0.6mm, F.Cu at (235.2, 88.7)
- added REF**: VIA-0.6mm, VIA-0.6mm, F.Cu at (178.2, 22.7)
- added REF**: VIA-0.6mm, VIA-0.6mm, F.Cu at (119.7, 104.2)
- added REF**: VIA-0.6mm, VIA-0.6mm, F.Cu at (197.2, 64.7)
- added REF**: VIA-0.6mm, VIA-0.6mm, F.Cu at (138.4, 100.9)
- added REF**: VIA-0.6mm, VIA-0.6mm, F.Cu at (128.5, 44.7)
- added REF**: VIA-0.6mm, VIA-0.6mm, F.Cu at (197.2, 83.7)
- added REF**: VIA-0.6mm, VIA-0.6mm, F.Cu at (152.5, 29.7)
- added REF**: VIA-0.6mm, VIA-0.6mm, F.Cu at (197.2, 26.7)
- added REF**: VIA-0.6mm, VIA-0.6mm, F.Cu at (109.9, 49.0)
- added REF**: VIA-0.6mm, VIA-0.6mm, F.Cu at (216.2, 30.2)
- added REF**: VIA-0.6mm, VIA-0.6mm, F.Cu at (178.2, 59.7)
- added REF**: VIA-0.6mm, VIA-0.6mm, F.Cu at (131.8, 63.4)
- added REF**: VIA-0.6mm, VIA-0.6mm, F.Cu at (178.2, 60.7)
- added _44: , R_0805_2012Metric_Pad1.20x1.40mm_HandSolder, F.Cu at (237.7, 68.0)
- added _44: , D_0805_2012Metric_Pad1.15x1.40mm_HandSolder, F.Cu at (237.7, 68.0)
- moved MH1 0.79 mm to (230.4, 82.7)
- moved MH2 0.44 mm to (253.4, 82.7)
- moved D4 0.33 mm to (138.7, 59.5)
- moved D26 0.33 mm to (242.7, 88.4)
- moved DISP1 0.33 mm to (237.7, 48.5)
- moved S26 0.33 mm to (235.2, 96.7)
- moved D7 0.33 mm to (185.7, 76.0)
- moved D8 0.33 mm to (185.7, 38.0)
- moved S1 0.33 mm to (121.0, 112.0)
- moved S15 0.33 mm to (178.2, 67.7)
- moved S24 0.33 mm to (216.2, 56.2)
- moved _43 0.33 mm to (251.4, 28.7)
- moved S9 0.33 mm to (158.0, 93.4)
- moved D11 0.33 mm to (223.7, 83.5)
- moved H3 0.33 mm to (211.0, 24.1)
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Routing:
- net GND: track 121.2 -> 109.4 mm
- net VCC: track 50.8 -> 41.0 mm, vias 0 -> 1
- net P2: track 50.4 -> 41.1 mm
- net RAW: track 25.5 -> 17.6 mm
- net P10: track 137.1 -> 144.7 mm
- net P3: track 40.1 -> 33.0 mm, vias 1 -> 2
- net P20: track 289.9 -> 296.0 mm
- net RST: track 41.7 -> 36.7 mm, vias 0 -> 1
- net P5: track 167.0 -> 171.2 mm
- net P19: track 268.9 -> 273.0 mm
- net P7: track 178.3 -> 182.1 mm
- net P1: track 70.9 -> 68.0 mm
- net P6: track 204.5 -> 207.3 mm
- net P15: track 251.1 -> 253.4 mm
- net P18: track 239.4 -> 241.5 mm
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Other:
- board text added: "Q'APLA"
